File: Mini_ELRS.kicad_sch (KiCad schematic)
At the start: 23 parts, among them J1 Conn_01x04, U1 ESP8266EX, U2 TC2014-3.3VxCTTR, U3 SX1280IMLTRT, Y1 52M, Y2 52M

Commit message: add motor and servo interface
Signed-off-by: huangzzk <huangcmzzk@gmail.com>
Parts:
- removed J1: Conn_01x04, Connector_PinHeader_2.54mm:PinHeader_1x04_P2.54mm_Vertical, symbol Connector_Generic:Conn_01x04
- removed TP1: TestPoint, TestPoint:TestPoint_Pad_1.0x1.0mm, symbol Connector:TestPoint
- added J1: Conn_01x05, Connector_PinHeader_2.54mm:PinHeader_1x05_P2.54mm_Vertical, symbol Connector_Generic:Conn_01x05
- added J2, J3: Conn_01x02_MountingPin, Connector_Molex:Molex_CLIK-Mate_502386-0270_1x02-1MP_P1.25mm_Horizontal, symbol Connector_Generic_MountingPin:Conn_01x02_MountingPin
- added J4, J6: Conn_01x03_MountingPin, Connector_Molex:Molex_CLIK-Mate_502386-0370_1x03-1MP_P1.25mm_Horizontal, symbol Connector_Generic_MountingPin:Conn_01x03_MountingPin
- added Q1, Q2: Q_NMOS_GSD, Package_TO_SOT_SMD:SOT-23, symbol Device:Q_NMOS_GSD
- added R2, R6: 10K, Resistor_SMD:R_0402_1005Metric, symbol Device:R
Connections:
- net +5V: now also J1.1 (Pin_1), J2.1 (Pin_1), J3.1 (Pin_1), J4.2 (Pin_2), J6.2 (Pin_2)
- net GND: now also J1.4 (Pin_4), J2.MP (MountPin), J3.MP (MountPin), J4.3 (Pin_3), J4.MP (MountPin), J6.3 (Pin_3), J6.MP (MountPin), Q1.2 (S), Q2.2 (S), R2.2, R6.2
- net RX: now also J1.2 (Pin_2)
- net TX: now also J1.3 (Pin_3)
- net GPIO0: now reaches U1.15 (GPIO0)
- net GPIO0: now also J1.5 (Pin_5)
- net PWM3: now reaches U1.18 (SDIO_DATA_2)
- net PWM3: now also Q1.1 (G), R2.1
- net PWM4: now reaches U1.19 (SDIO_DATA_3)
- net PWM4: now also J4.1 (Pin_1)
- net ANT: now reaches U1.2 (LNA)
- net PWM1: now reaches U1.20 (SDIO_CMD)
- net PWM1: now also J6.1 (Pin_1)
- net PWM2: now reaches U1.22 (SDIO_DATA_0)
- net PWM2: now also Q2.1 (G), R6.1
- new net: J3.2 (Pin_2), Q2.3 (D)
- new net: J2.2 (Pin_2), Q1.3 (D)
Other:
- moved on the sheet: C2, C4, U2

Commit message: fix wrong pwm pins
Signed-off-by: huangzzk <huangcmzzk@gmail.com>
Connections:
- net RX is gone; now on net PWM1: J1.2 (Pin_2), U1.25 (U0RXD)
- net BUSY: no longer U1.24 (GPIO5)
- net PWM1: no longer U1.20 (SDIO_CMD)
- net PWM2: now also U1.24 (GPIO5); no longer U1.22 (SDIO_DATA_0)
Other:
- note added: "RX GPIO3 SDIO_DATA2 GPIO9 SDIO_DATA3 GPIO10"
Changed lines of the file:
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@@
+    (stroke (width 0) (type default) (color 0 0 0 0))
+  )
+  (wire (pts (xy 89.535 73.025) (xy 94.615 73.025))
     (stroke (width 0) (type default) (color 0 0 0 0))
   )
@@
   (wire (pts (xy 29.21 76.2) (xy 29.21 75.565))
     (stroke (width 0) (type default) (color 0 0 0 0))
+  )
+  (text "RX GPIO3\nSDIO_DATA2 GPIO9\nSDIO_DATA3 GPIO10" (at 101.6 67.31 0)
+    (effects (font (size 1.27 1.27)) (justify left bottom))
   )
   (label "PWM3" (at 36.195 165.735 0)
@@
     (effects (font (size 1.27 1.27)) (justify right bottom))
   )
+  (label "PWM2" (at 89.535 88.265 0)
+    (effects (font (size 1.27 1.27)) (justify left bottom))
+  )
   (label "RF" (at 167.64 125.095 0)
-    (effects (font (size 1.27 1.27)) (justify left bottom))
-  )
-  (label "PWM1" (at 89.535 60.325 0)
     (effects (font (size 1.27 1.27)) (justify left bottom))
   )
@@
     (effects (font (size 1.27 1.27)) (justify right bottom))
   )
+  (label "PWM1" (at 94.615 73.025 0)
+    (effects (font (size 1.27 1.27)) (justify left bottom))
+  )
   (label "MOSI" (at 89.535 85.725 0)
     (effects (font (size 1.27 1.27)) (justify left bottom))
@@
     (effects (font (size 1.27 1.27)) (justify left bottom))
   )
-  (label "PWM2" (at 89.535 65.405 0)
-    (effects (font (size 1.27 1.27)) (justify left bottom))
-  )
   (label "PWM2" (at 80.01 167.005 0)
     (effects (font (size 1.27 1.27)) (justify left bottom))
@@
     (effects (font (size 1.27 1.27)) (justify left bottom))
   )
-  (label "BUSY" (at 89.535 88.265 0)
-    (effects (font (size 1.27 1.27)) (justify left bottom))
-  )

Commit message: update
Signed-off-by: huangzzk <huangcmzzk@gmail.com>
Parts:
- Y2: value 52M -> 26M
Connections:
- net DIO1: now also U1.18 (SDIO_DATA_2); no longer U1.16 (GPIO4)
- net PWM3: now also U1.16 (GPIO4); no longer U1.18 (SDIO_DATA_2)
Changed lines of the file:
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@@
+    (effects (font (size 1.27 1.27)) (justify left bottom))
+  )
+  (label "PWM3" (at 89.535 98.425 0)
     (effects (font (size 1.27 1.27)) (justify left bottom))
   )
@@
     (effects (font (size 1.27 1.27)) (justify left bottom))
   )
-  (label "DIO1" (at 89.535 98.425 0)
+  (label "DIO1" (at 89.535 67.945 0)
     (effects (font (size 1.27 1.27)) (justify left bottom))
   )
@@
   )
   (label "PWM4" (at 89.535 70.485 0)
-    (effects (font (size 1.27 1.27)) (justify left bottom))
-  )
-  (label "PWM3" (at 89.535 67.945 0)
     (effects (font (size 1.27 1.27)) (justify left bottom))
   )
@@
     (in_bom yes) (on_board yes)
     (property "Reference" "Y2" (id 0) (at 34.925 88.265 90))
-    (property "Value" "52M" (id 1) (at 33.655 92.71 90))
+    (property "Value" "26M" (id 1) (at 33.655 92.71 90))
     (property "Footprint" "Crystal:Crystal_SMD_2520-4Pin_2.5x2.0mm" (id 2) (at 37.465 91.44 0)
       (effects (font (size 1.27 1.27)) hide)
@@
     )
     (path "/6ceec7ee-4bcd-4970-abb4-553246f38eb5"
-      (reference "Y2") (unit 1) (value "52M") (footprint "Crystal:Crystal_SMD_2520-4Pin_2.5x2.0mm")
-    )
-  )
+      (reference "Y2") (unit 1) (value "26M") (footprint "Crystal:Crystal_SMD_2520-4Pin_2.5x2.0mm")
+    )
+  )

Commit message: update mcu to esp8285 rather than esp8266
Signed-off-by: huangzzk <huangcmzzk@gmail.com>
Parts:
- U1: value ESP8266EX -> ESP8285
Changed lines of the file:
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@@
   (symbol (lib_id "MCU_Espressif:ESP8266EX") (at 66.675 78.105 0) (unit 1)
     (in_bom yes) (on_board yes) (fields_autoplaced)
-    (property "Reference" "U1" (id 0) (at 68.6944 106.045 0)
-      (effects (font (size 1.27 1.27)) (justify left))
-    )
-    (property "Value" "ESP8266EX" (id 1) (at 68.6944 108.585 0)
+    (property "Reference" "U1" (id 0) (at 68.6944 106.68 0)
+      (effects (font (size 1.27 1.27)) (justify left))
+    )
+    (property "Value" "ESP8285" (id 1) (at 68.6944 109.22 0)
       (effects (font (size 1.27 1.27)) (justify left))
     )
@@
     )
     (path "/85e78923-8588-4c12-be82-1339495de1d9"
-      (reference "U1") (unit 1) (value "ESP8266EX") (footprint "Package_DFN_QFN:QFN-32-1EP_5x5mm_P0.5mm_EP3.45x3.45mm")
+      (reference "U1") (unit 1) (value "ESP8285") (footprint "Package_DFN_QFN:QFN-32-1EP_5x5mm_P0.5mm_EP3.45x3.45mm")
     )
     (path "/834aa2b6-a999-41a3-bbad-701366e676b1"

Commit message: v2.2 add diode in motor interface
Signed-off-by: huangzzk <huangcmzzk@gmail.com>
Parts:
- added D1, D3: D, Diode_SMD:D_SOD-323, symbol Device:D
Connections:
- net +5V: now also D1.1 (K), D3.1 (K)
- net at J3.2 (Pin_2), Q2.3 (D): now also D3.2 (A)
- net at J2.2 (Pin_2), Q1.3 (D): now also D1.2 (A)
Changed lines of the file:
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@@
   (junction (at 56.515 52.705) (diameter 0) (color 0 0 0 0)
   )
+  (junction (at 50.8 158.115) (diameter 0) (color 0 0 0 0)
+  )
   (junction (at 238.125 92.71) (diameter 0) (color 0 0 0 0)
   )
@@
   (junction (at 189.23 90.17) (diameter 0) (color 0 0 0 0)
   )
+  (junction (at 43.18 155.575) (diameter 0) (color 0 0 0 0)
+  )
   (junction (at 273.685 147.32) (diameter 0) (color 0 0 0 0)
   )
   (junction (at 255.27 157.48) (diameter 0) (color 0 0 0 0)
   )
+  (junction (at 94.615 159.385) (diameter 0) (color 0 0 0 0)
+  )
   (junction (at 43.18 165.735) (diameter 0) (color 0 0 0 0)
   )
   (junction (at 241.3 149.86) (diameter 0) (color 0 0 0 0)
+  )
+  (junction (at 86.995 156.845) (diameter 0) (color 0 0 0 0)
   )
   (junction (at 229.87 59.69) (diameter 0) (color 0 0 0 0)
@@
   (no_connect (at 194.31 85.09))
   (no_connect (at 229.87 87.63))
+  (wire (pts (xy 43.18 158.115) (xy 43.18 155.575))
+    (stroke (width 0) (type default) (color 0 0 0 0))
+  )
   (wire (pts (xy 161.29 152.4) (xy 167.64 152.4))
     (stroke (width 0) (type default) (color 0 0 0 0))
@@
     (stroke (width 0) (type default) (color 0 0 0 0))
   )
+  (wire (pts (xy 86.995 156.845) (xy 86.995 159.385))
+    (stroke (width 0) (type default) (color 0 0 0 0))
+  )
   (wire (pts (xy 234.95 147.32) (xy 241.3 147.32))
     (stroke (width 0) (type default) (color 0 0 0 0))
@@
     (stroke (width 0) (type default) (color 0 0 0 0))
   )
-  (wire (pts (xy 36.195 155.575) (xy 50.8 155.575))
+  (wire (pts (xy 36.195 155.575) (xy 43.18 155.575))
+    (stroke (width 0) (type default) (color 0 0 0 0))
+  )
+  (wire (pts (xy 86.995 156.845) (xy 94.615 156.845))
     (stroke (width 0) (type default) (color 0 0 0 0))
   )
@@
     (stroke (width 0) (type default) (color 0 0 0 0))
   )
-  (wire (pts (xy 80.01 156.845) (xy 94.615 156.845))
+  (wire (pts (xy 80.01 156.845) (xy 86.995 156.845))
     (stroke (width 0) (type default) (color 0 0 0 0))
   )
@@
   )
   (wire (pts (xy 37.465 85.725) (xy 37.465 88.9))
+    (stroke (width 0) (type default) (color 0 0 0 0))
+  )
+  (wire (pts (xy 43.18 155.575) (xy 50.8 155.575))
     (stroke (width 0) (type default) (color 0 0 0 0))
   )
@@
     )
     (pin "1")
+  )
+  (symbol (lib_id "Device:D") (at 46.99 158.115 0) (unit 1)
+    (in_bom yes) (on_board yes) (fields_autoplaced)
+    (property "Reference" "D1" (id 0) (at 46.99 151.765 0))
+    (property "Value" "D" (id 1) (at 46.99 154.305 0))
+    (property "Footprint" "Diode_SMD:D_SOD-323" (id 2) (at 46.99 158.115 0)
+      (effects (font (size 1.27 1.27)) hide)
+    )
+    (property "Datasheet" "~" (id 3) (at 46.99 158.115 0)
+      (effects (font (size 1.27 1.27)) hide)
+    )
+    (pin "1")
+    (pin "2")
   )
   (symbol (lib_id "Device:C") (at 238.125 88.9 0) (unit 1)
@@
     (pin "1")
   )
+  (symbol (lib_id "Device:D") (at 90.805 159.385 0) (unit 1)
+    (in_bom yes) (on_board yes) (fields_autoplaced)
+    (property "Reference" "D3" (id 0) (at 90.805 153.035 0))
+    (property "Value" "D" (id 1) (at 90.805 155.575 0))
+    (property "Footprint" "Diode_SMD:D_SOD-323" (id 2) (at 90.805 159.385 0)
+      (effects (font (size 1.27 1.27)) hide)
+    )
+    (property "Datasheet" "~" (id 3) (at 90.805 159.385 0)
+      (effects (font (size 1.27 1.27)) hide)
+    )
+    (pin "1")
+    (pin "2")
+  )
   (symbol (lib_id "power:GND") (at 160.02 157.48 0) (unit 1)
     (in_bom yes) (on_board yes) (fields_autoplaced)
@@
       (reference "C10") (unit 1) (value "0.1uF") (footprint "Capacitor_SMD:C_0402_1005Metric")
     )
+    (path "/1de863bb-d061-4f07-9051-fcd60169ad02"
+      (reference "D1") (unit 1) (value "D") (footprint "Diode_SMD:D_SOD-323")
+    )
     (path "/852fe9ae-45a6-469f-b59b-1795f0023edd"
       (reference "D2") (unit 1) (value "LED") (footprint "LED_SMD:LED_0603_1608Metric")
     )
+    (path "/a0c87b98-0335-47d5-aeec-4349b4ce187b"
+      (reference "D3") (unit 1) (value "D") (footprint "Diode_SMD:D_SOD-323")
+    )
     (path "/50d0a559-f09c-43ba-9759-3e2ba4b680a7"

Commit message: 3.0 add imu 42670
Signed-off-by: huangzzk <huangcmzzk@gmail.com>
Parts:
- added AE2: Antenna, Capacitor_SMD:C_1206_3216Metric, symbol Device:Antenna
- added I1: ICM20600, Package_LGA:Bosch_LGA-14_3x2.5mm_P0.5mm, symbol ic:ICM20600
- added R7, R8: 10K, Resistor_SMD:R_0402_1005Metric, symbol Device:R
Connections:
- net +3V3: now also I1.12 (nCS), I1.5 (VDD), I1.8 (VDD), R7.2, R8.2
- net GND: now also I1.1 (AD0), I1.6 (GND), I1.7 (REV)
- net GPIO0: now also I1.14 (SDA), R8.1
- net ANT: no longer names the net of U1.2 (LNA)
- net ANT: now also AE2.1 (A)
- net TX renamed SCL
- net SCL: now also I1.13 (SCL), R7.1
